File: scalenode-cm4-baseboard.kicad_sch (KiCad schematic)
At the start: 2 parts

Commit message: [#46875] kmake loclib
Parts:
- N1: footprint antmicro-footprints:antmicro-logo_scaled_15mm -> scalenode-cm4-baseboard-footprints:antmicro-logo_scaled_15mm; symbol antmicroMechanicalParts:antmicro_logo -> scalenode-cm4-baseboard:antmicro_logo
- N3: footprint antmicro-footprints:oshw-logo -> scalenode-cm4-baseboard-footprints:oshw-logo; symbol antmicroMechanicalParts:oshw_logo -> scalenode-cm4-baseboard:oshw_logo

Commit message: [#56969] Correct component references
Parts:
- N1: footprint scalenode-cm4-baseboard-footprints:antmicro-logo_scaled_15mm -> scalenode-cm4-baseboard-footprints:antmicro-logo
